File: audio_board/audio_board.sch (EAGLE design)
At the start: 20 parts

Commit message: audio board 01
Parts:
- removed BAT1: BAT_PAD, BAT_PAD:BAT_PAD
- removed BAT1_S: SWITCH_DPDT, ELEC327:SWITCH_DPDT
- removed BUTTON: (no value), switch-omron:10-XX
- removed C1: 470nf, rcl:C-USC1206
Connections:
- removed net BAT_VCC: BAT1.VDD, BAT1_S.2, BAT1_S.5
- removed net BTTN: BUTTON.S, BUTTON.S1, C1.1
- net GND: no longer BAT1.GND, BUTTON.P, BUTTON.P1, C1.2
- net VCC: no longer BAT1_S.1, BAT1_S.4
Other:
- moved on the sheet: C2, C3, C4, C6, R3, R4, R5, U$1

Commit message: finished audio board 1
Parts:
- added U$2: 1699_HEAD, 1699_Head:1699_HEAD
Connections:
- net GND: now also U$2.GND
- net L: now also U$2.ROUT
- net R: now also U$2.LOUT
Changed lines of the file:
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@@
 <?xml version="1.0" encoding="utf-8"?>
 <!DOCTYPE eagle SYSTEM "eagle.dtd">
-<eagle version="8.6.0">
+<eagle version="8.2.2">
 <drawing>
 <settings>
 <setting alwaysvectorfont="no"/>
-<setting keepoldvectorfont="yes"/>
 <setting verticaltext="up"/>
 </settings>
@@
 <part name="CSUPPLY3" library="rcl" deviceset="C-US" device="C1206" value="10uf"/>
 <part name="R2" library="resistor" library_urn="urn:adsk.eagle:library:348" deviceset="R-US_" device="R1206" value="47k"/>
-<part name="U$1" library="msgeq7" deviceset="MSGEQ7" device=""/>
 <part name="R3" library="resistor" library_urn="urn:adsk.eagle:library:348" deviceset="R-US_" device="R1206" value="22K"/>
 <part name="R4" library="resistor" library_urn="urn:adsk.eagle:library:348" deviceset="R-US_" device="R1206" value="22K"/>
@@
 <part name="GND8" library="supply1" deviceset="GND" device=""/>
 <part name="PWR_FED" library="pinhead" library_urn="urn:adsk.eagle:library:325" deviceset="PINHD-1X4" device=""/>
+<part name="U$2" library="1699_Head" deviceset="1699_HEAD" device=""/>
+<part name="GND2" library="supply1" deviceset="GND" device=""/>
+<part name="U$1" library="msgeq7" deviceset="MSGEQ7" device=""/>
 </parts>
 <sheets>
@@
 <instance part="CSUPPLY3" gate="G$1" x="-83.82" y="218.44"/>
 <instance part="R2" gate="G$1" x="-17.78" y="208.28" rot="R90"/>
-<instance part="U$1" gate="G$1" x="-116.84" y="137.16"/>
 <instance part="R3" gate="G$1" x="-81.28" y="149.86" rot="R180"/>
 <instance part="R4" gate="G$1" x="-81.28" y="142.24"/>
@@
 <instance part="GND8" gate="1" x="-147.32" y="137.16"/>
 <instance part="PWR_FED" gate="A" x="7.62" y="157.48"/>
+<instance part="U$2" gate="G$1" x="-55.88" y="144.78" rot="R90"/>
+<instance part="GND2" gate="1" x="-38.1" y="144.78" rot="R90"/>
+<instance part="U$1" gate="G$1" x="-116.84" y="137.16"/>
 </instances>
 <busses>
@@
 <segment>
 <pinref part="GND4" gate="1" pin="GND"/>
+<wire x1="-119.38" y1="109.22" x2="-119.38" y2="116.84" width="0.1524" layer="91"/>
 <pinref part="U$1" gate="G$1" pin="2"/>
-<wire x1="-119.38" y1="109.22" x2="-119.38" y2="116.84" width="0.1524" layer="91"/>
 </segment>
 <segment>
@@
 <wire x1="5.08" y1="154.94" x2="0" y2="154.94" width="0.1524" layer="91"/>
 <label x="-2.54" y="154.94" size="1.778" layer="95"/>
+</segment>
+<segment>
+<pinref part="U$2" gate="G$1" pin="GND"/>
+<pinref part="GND2" gate="1" pin="GND"/>
+<wire x1="-48.26" y1="144.78" x2="-40.64" y2="144.78" width="0.1524" layer="91"/>
 </segment>
 </net>
@@
 <segment>
 <pinref part="P+3" gate="VCC" pin="VCC"/>
-<pinref part="U$1" gate="G$1" pin="1"/>
 <wire x1="-124.46" y1="104.14" x2="-124.46" y2="109.22" width="0.1524" layer="91"/>
 <pinref part="C2" gate="G$1" pin="1"/>
@@
 <wire x1="-134.62" y1="109.22" x2="-124.46" y2="109.22" width="0.1524" layer="91"/>
 <junction x="-124.46" y="109.22"/>
+<pinref part="U$1" gate="G$1" pin="1"/>
 </segment>
 <segment>
@@
 </segment>
 <segment>
-<pinref part="U$1" gate="G$1" pin="7"/>
 <wire x1="-119.38" y1="144.78" x2="-119.38" y2="149.86" width="0.1524" layer="91"/>
 <label x="-119.38" y="149.86" size="1.778" layer="95" rot="R90"/>
+<pinref part="U$1" gate="G$1" pin="7"/>
 </segment>
 </net>
@@
 </segment>
 <segment>
-<pinref part="U$1" gate="G$1" pin="3"/>
 <wire x1="-114.3" y1="116.84" x2="-114.3" y2="114.3" width="0.1524" layer="91"/>
 <label x="-114.3" y="114.3" size="1.778" layer="95" rot="R270"/>
+<pinref part="U$1" gate="G$1" pin="3"/>
 </segment>
 </net>
@@
 </segment>
 <segment>
-<pinref part="U$1" gate="G$1" pin="4"/>
 <wire x1="-109.22" y1="116.84" x2="-109.22" y2="111.76" width="0.1524" layer="91"/>
 <label x="-109.22" y="111.76" size="1.778" layer="95" rot="R270"/>
+<pinref part="U$1" gate="G$1" pin="4"/>
 </segment>
 </net>
 <net name="N$1" class="0">
 <segment>
-<pinref part="U$1" gate="G$1" pin="5"/>
 <wire x1="-109.22" y1="144.78" x2="-109.22" y2="149.86" width="0.1524" layer="91"/>
 <pinref part="C3" gate="G$1" pin="2"/>
 <wire x1="-109.22" y1="149.86" x2="-99.06" y2="149.86" width="0.1524" layer="91"/>
+<pinref part="U$1" gate="G$1" pin="5"/>
 </segment>
 </net>
@@
 <wire x1="-76.2" y1="149.86" x2="-71.12" y2="149.86" width="0.1524" layer="91"/>
 <label x="-71.12" y="149.86" size="1.778" layer="95"/>
+<pinref part="U$2" gate="G$1" pin="ROUT"/>
+<wire x1="-66.04" y1="152.4" x2="-71.12" y2="152.4" width="0.1524" layer="91"/>
+<wire x1="-71.12" y1="152.4" x2="-71.12" y2="149.86" width="0.1524" layer="91"/>
 </segment>
 </net>
@@
 <wire x1="-76.2" y1="142.24" x2="-71.12" y2="142.24" width="0.1524" layer="91"/>
 <label x="-71.12" y="142.24" size="1.778" layer="95"/>
+<pinref part="U$2" gate="G$1" pin="LOUT"/>
+<wire x1="-66.04" y1="139.7" x2="-71.12" y2="139.7" width="0.1524" layer="91"/>
+<wire x1="-71.12" y1="139.7" x2="-71.12" y2="142.24" width="0.1524" layer="91"/>
 </segment>
 </net>
@@
 <segment>
 <pinref part="C6" gate="G$1" pin="2"/>
+<wire x1="-114.3" y1="149.86" x2="-114.3" y2="144.78" width="0.1524" layer="91"/>
 <pinref part="U$1" gate="G$1" pin="6"/>
-<wire x1="-114.3" y1="149.86" x2="-114.3" y2="144.78" width="0.1524" layer="91"/>
 </segment>
 </net>
 <net name="N$4" class="0">
 <segment>
-<pinref part="U$1" gate="G$1" pin="8"/>
 <wire x1="-124.46" y1="144.78" x2="-124.46" y2="154.94" width="0.1524" layer="91"/>
 <pinref part="R5" gate="G$1" pin="2"/>
@@
 <wire x1="-147.32" y1="154.94" x2="-137.16" y2="154.94" width="0.1524" layer="91"/>
 <junction x="-137.16" y="154.94"/>
+<pinref part="U$1" gate="G$1" pin="8"/>
 </segment>
 </net>
@@
 <compatibility>
 <note version="8.2" severity="warning">
-Since Version 8.2, EAGLE supports online libraries. The ids
+Since Version 8.2, Eagle supports online libraries. The ids
 of those online libraries will not be understood (or retained)
 with this version.
